File: Kicad/ZPE Atom controller/ZPE Atom controller.kicad_sch (KiCad schematic)
At the start: 24 parts, among them J1 50 ohm 21 turns, Q1 PN2222A, Q2 IRFZ44N, SW1 ON/OFF, T1 Transformer_SP_1S, U2 LM7805_TO220

Commit message: Added new Kicad files
Parts:
- added P1, P2: CONN_01X18, Connector_PinHeader_2.54mm:PinHeader_1x19_P2.54mm_Vertical, symbol Hornbill-Devboard-rescue:CONN_01X19
- added RV1, RV2: 10K, symbol Device:R_Potentiometer
- added RV3: 10k, symbol Device:R_Potentiometer
- added U1: SSD1306, Package_TO_SOT_SMD:SOT-23-5, symbol Memory_EEPROM:24AA02-OT
- T1: footprint (none) -> Transformer_THT:Transformer_NF_ETAL_P1165
Connections:
- net +5V: now also P1.19 (P19)
- net GND: now also P1.14 (P14), P2.7 (P7), RV1.3, RV2.3, RV3.3, U1.1 (GND)
- new net +3V3: RV1.1, RV2.1, RV3.1, U1.2 (VCC)
- new net CLK: P2.19 (P19)
- new net CMD: P1.18 (P18)
- new net EN: P1.2 (P2)
- new net IO0: P2.14 (P14)
- new net IO12: P1.13 (P13)
- new net IO13: P1.15 (P15)
- new net IO14: P1.12 (P12)
- new net IO15: P2.16 (P16)
- new net IO16: P2.12 (P12)
- new net IO17: P2.11 (P11)
- new net IO18: P2.9 (P9)
- new net IO19: P2.8 (P8)
- new net IO2: P2.15 (P15)
- new net IO21: P2.6 (P6), U1.3 (SCL)
- new net IO22: P2.3 (P3), U1.4 (SDA)
- new net IO23: P2.2 (P2)
- new net IO25: P1.9 (P9)
- new net IO26: P1.10 (P10)
- new net IO27: P1.11 (P11)
- new net IO32: P1.7 (P7)
- new net IO33: P1.8 (P8)
- new net IO34: P1.5 (P5), RV3.2
- new net IO35: P1.6 (P6), RV2.2
- new net IO36: P1.3 (P3), RV1.2
- new net IO39: P1.4 (P4)
- new net IO4: P2.13 (P13)
- new net IO5: P2.10 (P10)
- new net RXD0: P2.5 (P5)
- new net SD0: P2.18 (P18)
- new net SD1: P2.17 (P17)
- new net SD2: P1.16 (P16)
- new net SD3: P1.17 (P17)
- new net TXD0: P2.4 (P4)
Other:
- moved on the sheet: C1, C2, C3, C4, C5, C6, D1, D2, D3, D4, D5, J1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

Commit message: Working freq generator from 1 till 39mHZ
Parts:
- removed Q1: PN2222A, Package_TO_SOT_THT:TO-92_Inline, symbol Transistor_BJT:PN2222A
- removed R2: 1K, Resistors_THT:R_Axial_DIN0204_L3.6mm_D1.6mm_P7.62mm_Horizontal, symbol ZPE-test-3-small-board-only-rescue:R-device
Connections:
- net GND: now also Q2.3 (S)
- net at R1.1: now also Q2.1 (G)
Other:
- moved on the sheet: L1, L2, L3, L4, R1

Commit message: Updated schematic for 5 pots
Parts:
- added DutyCycle: 10k, symbol Device:R_Potentiometer
- added Resolution: 10K, symbol Device:R_Potentiometer
- renumbered RV2 to Freq_fine1, RV1 to Freq_rough1, RV3 to Freq_super_fine
Connections:
- net +3V3: now also DutyCycle.1, Resolution.1
- net GND: now also DutyCycle.3, Resolution.3
- net IO32: now also Freq_fine1.2
- net IO33: now also R1.2
- net IO34: now also Resolution.2; no longer Freq_super_fine.2
- net IO35: now also DutyCycle.2; no longer Freq_fine1.2
- net IO36: now also Freq_super_fine.2; no longer Freq_rough1.2
- net IO39: now also Freq_rough1.2
Other:
- moved on the sheet: L1, L2, L3, L4, P1, P2, U1

Commit message: Updated schematic
Parts:
- renumbered Freq_fine1 to Freq_fine, Freq_rough1 to Freq_rough
Other:
- moved on the sheet: Freq_fine, Freq_rough, L1, L2, L3, L4

Commit message: Updated board
Parts:
- added R2: 100k, Resistors_THT:R_Axial_DIN0204_L3.6mm_D1.6mm_P7.62mm_Horizontal, symbol ZPE-test-3-small-board-only-rescue:R-device
- R1: value 10k -> 1k
- renumbered DutyCycle to DutyCycle1, Freq_fine to Freq_fine1, Freq_rough to Freq_rough1, Freq_super_fine to Freq_super_fine1, Resolution to Resolution1
Connections:
- net +12V: now also R2.1
- net at Q2.1 (G), R1.1: now also R2.2
Changed lines of the file:
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@@
   (junction (at 162.56 45.085) (diameter 0) (color 0 0 0 0)
   )
+  (junction (at 150.495 42.545) (diameter 0) (color 0 0 0 0)
+  )
+  (junction (at 150.495 65.405) (diameter 0) (color 0 0 0 0)
+  )
   (junction (at 26.67 55.245) (diameter 0) (color 0 0 0 0)
   )
@@
     (stroke (width 0) (type default))
   )
+  (wire (pts (xy 150.495 65.405) (xy 154.94 65.405))
+    (stroke (width 0) (type default))
+  )
   (wire (pts (xy 196.85 128.905) (xy 191.77 128.905))
     (stroke (width 0) (type default))
@@
     (stroke (width 0) (type default))
   )
+  (wire (pts (xy 150.495 42.545) (xy 150.495 50.165))
+    (stroke (width 0) (type default))
+  )
   (wire (pts (xy 191.77 133.985) (xy 191.77 128.905))
     (stroke (width 0) (type default))
@@
     (stroke (width 0) (type default))
   )
-  (wire (pts (xy 154.94 65.405) (xy 150.495 65.405))
-    (stroke (width 0) (type default))
-  )
   (wire (pts (xy 41.656 89.535) (xy 37.846 89.535))
     (stroke (width 0) (type default))
@@
     (stroke (width 0) (type default))
   )
+  (wire (pts (xy 150.495 57.785) (xy 150.495 65.405))
+    (stroke (width 0) (type default))
+  )
   (wire (pts (xy 170.18 112.395) (xy 158.75 112.395))
     (stroke (width 0) (type default))
@@
     (stroke (width 0) (type default))
   )
+  (wire (pts (xy 150.495 42.545) (xy 162.56 42.545))
+    (stroke (width 0) (type default))
+  )
   (wire (pts (xy 54.61 64.77) (xy 52.07 64.77))
     (stroke (width 0) (type default))
@@
     (stroke (width 0) (type default))
   )
-  (wire (pts (xy 147.32 42.545) (xy 162.56 42.545))
+  (wire (pts (xy 147.32 42.545) (xy 150.495 42.545))
     (stroke (width 0) (type default))
   )
@@
   (symbol (lib_name "R_Potentiometer_3") (lib_id "Device:R_Potentiometer") (at 26.67 64.77 0) (unit 1)
     (in_bom yes) (on_board yes)
-    (property "Reference" "Freq_rough" (id 0) (at 32.639 69.342 0)
-      (effects (font (size 1.27 1.27)) (justify right))
-    )
-    (property "Value" "10K" (id 1) (at 24.13 63.5 90)
+    (property "Reference" "Freq_rough1" (id 0) (at 32.639 69.342 0)
+      (effects (font (size 1.27 1.27)) (justify right))
+    )
+    (property "Value" "10K" (id 1) (at 24.13 62.865 90)
       (effects (font (size 1.27 1.27)) (justify right))
     )
@@
   (symbol (lib_name "R_Potentiometer_2") (lib_id "Device:R_Potentiometer") (at 37.846 64.77 0) (unit 1)
     (in_bom yes) (on_board yes)
-    (property "Reference" "Freq_fine" (id 0) (at 43.434 69.596 0)
-      (effects (font (size 1.27 1.27)) (justify right))
-    )
-    (property "Value" "10K" (id 1) (at 35.306 63.5 90)
+    (property "Reference" "Freq_fine1" (id 0) (at 43.434 69.596 0)
+      (effects (font (size 1.27 1.27)) (justify right))
+    )
+    (property "Value" "10K" (id 1) (at 35.56 62.865 90)
       (effects (font (size 1.27 1.27)) (justify right))
     )
@@
   (symbol (lib_id "Device:R_Potentiometer") (at 48.895 81.28 0) (unit 1)
     (in_bom yes) (on_board yes)
-    (property "Reference" "DutyCycle" (id 0) (at 54.102 85.852 0)
+    (property "Reference" "DutyCycle1" (id 0) (at 54.102 85.852 0)
       (effects (font (size 1.27 1.27)) (justify right))
     )
@@
   (symbol (lib_name "R_Potentiometer_4") (lib_id "Device:R_Potentiometer") (at 37.846 81.28 0) (unit 1)
     (in_bom yes) (on_board yes)
-    (property "Reference" "Resolution" (id 0) (at 43.434 85.852 0)
+    (property "Reference" "Resolution1" (id 0) (at 43.434 85.852 0)
       (effects (font (size 1.27 1.27)) (justify right))
     )
@@
     (pin "2")
     (pin "3")
+  )
+  (symbol (lib_id "ZPE-test-3-small-board-only-rescue:R-device") (at 150.495 53.975 0) (unit 1)
+    (in_bom yes) (on_board yes)
+    (property "Reference" "R2" (id 0) (at 149.225 48.895 0)
+      (effects (font (size 1.27 1.27)))
+    )
+    (property "Value" "100k" (id 1) (at 150.495 53.975 90)
+      (effects (font (size 1.27 1.27)))
+    )
+    (property "Footprint" "Resistors_THT:R_Axial_DIN0204_L3.6mm_D1.6mm_P7.62mm_Horizontal" (id 2) (at 148.717 53.975 90)
+      (effects (font (size 1.27 1.27)) hide)
+    )
+    (property "Datasheet" "" (id 3) (at 150.495 53.975 0)
+      (effects (font (size 1.27 1.27)) hide)
+    )
+    (pin "1")
+    (pin "2")
   )
   (symbol (lib_id "Hornbill-Devboard-rescue:+3.3V") (at 126.365 85.09 0) (unit 1)
@@
       (effects (font (size 1.27 1.27)))
     )
-    (property "Value" "10k" (id 1) (at 143.51 72.39 90)
+    (property "Value" "1k" (id 1) (at 143.51 72.39 90)
       (effects (font (size 1.27 1.27)))
     )
@@
   (symbol (lib_name "R_Potentiometer_1") (lib_id "Device:R_Potentiometer") (at 48.26 64.77 0) (unit 1)
     (in_bom yes) (on_board yes)
-    (property "Reference" "Freq_super_fine" (id 0) (at 58.674 69.596 0)
-      (effects (font (size 1.27 1.27)) (justify right))
-    )
-    (property "Value" "10k" (id 1) (at 43.18 63.5 90)
+    (property "Reference" "Freq_super_fine1" (id 0) (at 58.674 69.596 0)
+      (effects (font (size 1.27 1.27)) (justify right))
+    )
+    (property "Value" "10k" (id 1) (at 45.72 62.865 90)
       (effects (font (size 1.27 1.27)) (justify right))
     )
@@
     )
     (path "/8d318414-9517-4202-915f-0b5ef6b7ee7b"
-      (reference "DutyCycle") (unit 1) (value "10k") (footprint "")
+      (reference "DutyCycle1") (unit 1) (value "10k") (footprint "")
     )
     (path "/418e19cf-ec07-4213-bdc9-0796888f3d79"
-      (reference "Freq_fine") (unit 1) (value "10K") (footprint "")
+      (reference "Freq_fine1") (unit 1) (value "10K") (footprint "")
     )
     (path "/3cf7e9c3-7cb7-4599-9fbc-80b563294a59"
-      (reference "Freq_rough") (unit 1) (value "10K") (footprint "")
+      (reference "Freq_rough1") (unit 1) (value "10K") (footprint "")
     )
     (path "/d0da5fea-7bb8-466a-808d-a285a956d318"
-      (reference "Freq_super_fine") (unit 1) (value "10k") (footprint "")
+      (reference "Freq_super_fine1") (unit 1) (value "10k") (footprint "")
     )
     (path "/9242e0f9-861b-4075-b6d9-7e339b399019"
@@
     )
     (path "/c93ffc52-1a01-4ad9-966c-ca8653297ccc"
-      (reference "R1") (unit 1) (value "10k") (footprint "Resistors_THT:R_Axial_DIN0204_L3.6mm_D1.6mm_P7.62mm_Horizontal")
+      (reference "R1") (unit 1) (value "1k") (footprint "Resistors_THT:R_Axial_DIN0204_L3.6mm_D1.6mm_P7.62mm_Horizontal")
+    )
+    (path "/b55f6fd6-b5a9-46c1-9ccf-a9b9dbedb0ae"
+      (reference "R2") (unit 1) (value "100k") (footprint "Resistors_THT:R_Axial_DIN0204_L3.6mm_D1.6mm_P7.62mm_Horizontal")
     )
     (path "/b363d91d-fcd7-4752-acfe-6ce43382c232"
-      (reference "Resolution") (unit 1) (value "10K") (footprint "")
+      (reference "Resolution1") (unit 1) (value "10K") (footprint "")
     )
     (path "/705edee1-fc19-4950-8aac-33bef617012c"

Commit message: Updated code
Parts:
- Q2: value IRFZ44N -> IRF510
Other:
- moved on the sheet: L1, L2, L3, L4
Changed lines of the file:
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@@
     (effects (font (size 1.27 1.27)) (justify left bottom))
   )
-  (text "Drift Step Recovery Diode info \nModel 2D524A/KD524A\n\nMaximum operating frequency     100GHz\nSwitching-off time                200ps\nMinority Carrier Lifetime           25ns\nRecovery Сharge                   250nC\nTerminal Capacitance (UR = 0V)   1.2pF\nTerminal Capacitance (UR = 6V)   0.2pF\nCase Capacitance                  0.2pF\nTerminal Inductance                0.7nH\nForward Voltage                    1V\nReverce Voltage                    24V\nForward Current                    40mA\nForward Current Pulse              400mA\nReverce Current                    2mA\nReverce Current  Pulce             0.6A\nPower dissipation                   200 mW\nTemperature range                 -60...+125 C"
+  (text "Drift Step Recovery Diode info \nModel 2D524A/KD524A\n\nMaximum operating frequency     100GHz\nSwitching-off time                200ps\nMinority Carrier Lifetime           25ns\nRecovery Сharge                   250nC\nTerminal Capacitance (UR = 0V)   1.2pF\nTerminal Capacitance (UR = 6V)   0.2pF\nCase Capacitance                  0.2pF\nTerminal Inductance                0.7nH\nForward Voltage                    1V\nReverce Voltage                    24V\nForward Current                    40mA\nForward Current Pulse              400mA\nReverce Current                    2mA\nReverce Current  Pulse             0.6A\nPower dissipation                   200 mW\nTemperature range                 -60...+125 C"
     (at 222.885 73.025 0)
     (effects (font (size 1.27 1.27)) (justify left bottom))
@@
   (symbol (lib_name "R_Potentiometer_3") (lib_id "Device:R_Potentiometer") (at 26.67 64.77 0) (unit 1)
     (in_bom yes) (on_board yes)
-    (property "Reference" "Freq_rough1" (id 0) (at 32.639 69.342 0)
+    (property "Reference" "Freq_rough1" (id 0) (at 22.225 59.055 90)
       (effects (font (size 1.27 1.27)) (justify right))
     )
@@
   (symbol (lib_name "R_Potentiometer_2") (lib_id "Device:R_Potentiometer") (at 37.846 64.77 0) (unit 1)
     (in_bom yes) (on_board yes)
-    (property "Reference" "Freq_fine1" (id 0) (at 43.434 69.596 0)
+    (property "Reference" "Freq_fine1" (id 0) (at 33.02 60.325 90)
       (effects (font (size 1.27 1.27)) (justify right))
     )
@@
   (symbol (lib_name "R_Potentiometer_1") (lib_id "Device:R_Potentiometer") (at 48.26 64.77 0) (unit 1)
     (in_bom yes) (on_board yes)
-    (property "Reference" "Freq_super_fine1" (id 0) (at 58.674 69.596 0)
+    (property "Reference" "Freq_super_fine1" (id 0) (at 43.815 56.515 90)
       (effects (font (size 1.27 1.27)) (justify right))
     )
@@
       (effects (font (size 1.27 1.27)) (justify left))
     )
-    (property "Value" "IRFZ44N" (id 1) (at 151.13 61.595 0)
+    (property "Value" "IRF510" (id 1) (at 151.13 61.595 0)
       (effects (font (size 1.27 1.27)) (justify left))
     )
@@
       (effects (font (size 1.27 1.27) italic) (justify left) hide)
     )
-    (property "Datasheet" "http://www.fairchildsemi.com/ds/BU/BUZ11.pdf" (id 3) (at 160.02 65.405 0)
+    (property "Datasheet" "https://www.jameco.com/Jameco/Products/ProdDS/209234FSC.pdf" (id 3) (at 160.02 65.405 0)
       (effects (font (size 1.27 1.27)) (justify left) hide)
     )
@@
     )
     (path "/eec6f1b0-e4aa-49f8-b4a3-e9424cd19e76"
-      (reference "Q2") (unit 1) (value "IRFZ44N") (footprint "Housings_SIP:SIP3_11.6x8.5mm")
+      (reference "Q2") (unit 1) (value "IRF510") (footprint "Housings_SIP:SIP3_11.6x8.5mm")
     )
     (path "/c93ffc52-1a01-4ad9-966c-ca8653297ccc"

Commit message: added resistor for mosfet
Parts:
- added Q1: Q_PNP_ECB, symbol Device:Q_PNP_ECB
- added R3: 4.7k, Resistors_THT:R_Axial_DIN0204_L3.6mm_D1.6mm_P7.62mm_Horizontal, symbol ZPE-test-3-small-board-only-rescue:R-device
Connections:
- net GND: now also Q1.2 (C), R3.2
- net at Q2.1 (G), R2.2: now also Q1.1 (E), R3.1; no longer R1.1
- new net: Q1.3 (B), R1.1
Other:
- moved on the sheet: R1
Changed lines of the file:
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@@
   (junction (at 150.495 42.545) (diameter 0) (color 0 0 0 0)
   )
+  (junction (at 154.305 65.405) (diameter 0) (color 0 0 0 0)
+  )
+  (junction (at 26.67 55.245) (diameter 0) (color 0 0 0 0)
+  )
+  (junction (at 191.77 123.825) (diameter 0) (color 0 0 0 0)
+  )
   (junction (at 150.495 65.405) (diameter 0) (color 0 0 0 0)
   )
-  (junction (at 26.67 55.245) (diameter 0) (color 0 0 0 0)
-  )
-  (junction (at 191.77 123.825) (diameter 0) (color 0 0 0 0)
-  )
   (junction (at 209.55 128.905) (diameter 0) (color 0 0 0 0)
   )
@@
     (stroke (width 0) (type default))
   )
-  (wire (pts (xy 147.32 72.39) (xy 150.495 72.39))
-    (stroke (width 0) (type default))
-  )
   (wire (pts (xy 120.015 87.63) (xy 131.445 87.63))
     (stroke (width 0) (type default))
@@
     (stroke (width 0) (type default))
   )
-  (wire (pts (xy 150.495 65.405) (xy 154.94 65.405))
+  (wire (pts (xy 150.495 65.405) (xy 154.305 65.405))
     (stroke (width 0) (type default))
   )
@@
     (stroke (width 0) (type default))
   )
+  (wire (pts (xy 145.415 72.39) (xy 145.415 65.405))
+    (stroke (width 0) (type default))
+  )
   (wire (pts (xy 41.656 89.535) (xy 37.846 89.535))
     (stroke (width 0) (type default))
@@
     (stroke (width 0) (type default))
   )
+  (wire (pts (xy 145.415 65.405) (xy 150.495 65.405))
+    (stroke (width 0) (type default))
+  )
   (wire (pts (xy 134.62 125.095) (xy 151.13 125.095))
     (stroke (width 0) (type default))
@@
     (stroke (width 0) (type default))
   )
-  (wire (pts (xy 125.73 50.165) (xy 125.73 72.39))
+  (wire (pts (xy 125.73 50.165) (xy 125.73 77.47))
+    (stroke (width 0) (type default))
+  )
+  (wire (pts (xy 154.305 65.405) (xy 154.94 65.405))
     (stroke (width 0) (type default))
   )
@@
     (stroke (width 0) (type default))
   )
+  (wire (pts (xy 154.305 69.215) (xy 154.305 65.405))
+    (stroke (width 0) (type default))
+  )
   (wire (pts (xy 187.96 45.085) (xy 198.12 45.085))
     (stroke (width 0) (type default))
@@
     (stroke (width 0) (type default))
   )
-  (wire (pts (xy 125.73 72.39) (xy 139.7 72.39))
-    (stroke (width 0) (type default))
-  )
   (wire (pts (xy 55.245 67.31) (xy 73.025 67.31))
     (stroke (width 0) (type default))
@@
     (stroke (width 0) (type default))
   )
-  (wire (pts (xy 150.495 65.405) (xy 150.495 72.39))
-    (stroke (width 0) (type default))
-  )
   (wire (pts (xy 204.47 133.985) (xy 209.55 133.985))
     (stroke (width 0) (type default))
@@
   )
   (wire (pts (xy 55.245 67.31) (xy 55.245 81.28))
+    (stroke (width 0) (type default))
+  )
+  (wire (pts (xy 125.73 77.47) (xy 130.175 77.47))
     (stroke (width 0) (type default))
   )
@@
     (pin "2")
   )
+  (symbol (lib_id "power:GND") (at 145.415 82.55 0) (unit 1)
+    (in_bom yes) (on_board yes) (fields_autoplaced)
+    (property "Reference" "#PWR07" (id 0) (at 145.415 88.9 0)
+      (effects (font (size 1.27 1.27)) hide)
+    )
+    (property "Value" "GND" (id 1) (at 145.415 87.63 0)
+      (effects (font (size 1.27 1.27)))
+    )
+    (property "Footprint" "" (id 2) (at 145.415 82.55 0)
+      (effects (font (size 1.27 1.27)) hide)
+    )
+    (property "Datasheet" "" (id 3) (at 145.415 82.55 0)
+      (effects (font (size 1.27 1.27)) hide)
+    )
+    (pin "1")
+  )
   (symbol (lib_id "Device:Lamp") (at 200.66 150.495 90) (unit 1)
     (in_bom yes) (on_board yes)
@@
     (pin "1")
     (pin "2")
+  )
+  (symbol (lib_id "power:GND") (at 154.305 76.835 0) (unit 1)
+    (in_bom yes) (on_board yes) (fields_autoplaced)
+    (property "Reference" "#PWR08" (id 0) (at 154.305 83.185 0)
+      (effects (font (size 1.27 1.27)) hide)
+    )
+    (property "Value" "GND" (id 1) (at 154.305 81.915 0)
+      (effects (font (size 1.27 1.27)))
+    )
+    (property "Footprint" "" (id 2) (at 154.305 76.835 0)
+      (effects (font (size 1.27 1.27)) hide)
+    )
+    (property "Datasheet" "" (id 3) (at 154.305 76.835 0)
+      (effects (font (size 1.27 1.27)) hide)
+    )
+    (pin "1")
   )
   (symbol (lib_id "Hornbill-Devboard-rescue:+3.3V") (at 26.67 55.245 0) (unit 1)
@@
     (pin "2")
   )
+  (symbol (lib_id "ZPE-test-3-small-board-only-rescue:R-device") (at 154.305 73.025 0) (unit 1)
+    (in_bom yes) (on_board yes)
+    (property "Reference" "R3" (id 0) (at 153.035 67.945 0)
+      (effects (font (size 1.27 1.27)))
+    )
+    (property "Value" "4.7k" (id 1) (at 154.305 73.025 90)
+      (effects (font (size 1.27 1.27)))
+    )
+    (property "Footprint" "Resistors_THT:R_Axial_DIN0204_L3.6mm_D1.6mm_P7.62mm_Horizontal" (id 2) (at 152.527 73.025 90)
+      (effects (font (size 1.27 1.27)) hide)
+    )
+    (property "Datasheet" "" (id 3) (at 154.305 73.025 0)
+      (effects (font (size 1.27 1.27)) hide)
+    )
+    (pin "1")
+    (pin "2")
+  )
   (symbol (lib_id "Device:Transformer_SP_1S") (at 177.8 50.165 0) (unit 1)
     (in_bom yes) (on_board yes) (fields_autoplaced)
@@
     (pin "1")
   )
+  (symbol (lib_id "Device:Q_PNP_ECB") (at 142.875 77.47 0) (mirror x) (unit 1)
+    (in_bom yes) (on_board yes)
+    (property "Reference" "Q1" (id 0) (at 148.59 76.835 0)
+      (effects (font (size 1.27 1.27)) (justify left))
+    )
+    (property "Value" "Q_PNP_ECB" (id 1) (at 133.35 82.55 0)
+      (effects (font (size 1.27 1.27)) (justify left))
+    )
+    (property "Footprint" "" (id 2) (at 147.955 80.01 0)
+      (effects (font (size 1.27 1.27)) hide)
+    )
+    (property "Datasheet" "~" (id 3) (at 142.875 77.47 0)
+      (effects (font (size 1.27 1.27)) hide)
+    )
+    (pin "1")
+    (pin "2")
+    (pin "3")
+  )
   (symbol (lib_id "power:Earth") (at 184.15 117.475 0) (unit 1)
     (in_bom yes) (on_board yes) (fields_autoplaced)
@@
     (pin "2")
   )
-  (symbol (lib_id "ZPE-test-3-small-board-only-rescue:R-device") (at 143.51 72.39 270) (unit 1)
-    (in_bom yes) (on_board yes)
-    (property "Reference" "R1" (id 0) (at 148.59 71.12 90)
-      (effects (font (size 1.27 1.27)))
-    )
-    (property "Value" "1k" (id 1) (at 143.51 72.39 90)
-      (effects (font (size 1.27 1.27)))
-    )
-    (property "Footprint" "Resistors_THT:R_Axial_DIN0204_L3.6mm_D1.6mm_P7.62mm_Horizontal" (id 2) (at 143.51 70.612 90)
-      (effects (font (size 1.27 1.27)) hide)
-    )
-    (property "Datasheet" "" (id 3) (at 143.51 72.39 0)
+  (symbol (lib_id "ZPE-test-3-small-board-only-rescue:R-device") (at 133.985 77.47 270) (unit 1)
+    (in_bom yes) (on_board yes)
+    (property "Reference" "R1" (id 0) (at 139.065 76.2 90)
+      (effects (font (size 1.27 1.27)))
+    )
+    (property "Value" "1k" (id 1) (at 133.985 77.47 90)
+      (effects (font (size 1.27 1.27)))
+    )
+    (property "Footprint" "Resistors_THT:R_Axial_DIN0204_L3.6mm_D1.6mm_P7.62mm_Horizontal" (id 2) (at 133.985 75.692 90)
+      (effects (font (size 1.27 1.27)) hide)
+    )
+    (property "Datasheet" "" (id 3) (at 133.985 77.47 0)
       (effects (font (size 1.27 1.27)) hide)
     )
@@
       (reference "#PWR06") (unit 1) (value "Earth") (footprint "")
     )
+    (path "/07fc543e-ebc7-4da4-ab80-a5a9d1298f42"
+      (reference "#PWR07") (unit 1) (value "GND") (footprint "")
+    )
+    (path "/1a3c0592-bae7-4dc8-bfdf-de050749f428"
+      (reference "#PWR08") (unit 1) (value "GND") (footprint "")
+    )
     (path "/beea61b7-6b97-4cff-b7b6-f7b521c060b1"
       (reference "#PWR0101") (unit 1) (value "Earth") (footprint "")
@@
       (reference "P2") (unit 1) (value "CONN_01X18") (footprint "Connector_PinHeader_2.54mm:PinHeader_1x19_P2.54mm_Vertical")
     )
+    (path "/bba52ae1-2c60-4612-b640-b785ed4cdd7e"
+      (reference "Q1") (unit 1) (value "Q_PNP_ECB") (footprint "")
+    )
     (path "/eec6f1b0-e4aa-49f8-b4a3-e9424cd19e76"
       (reference "Q2") (unit 1) (value "IRF510") (footprint "Housings_SIP:SIP3_11.6x8.5mm")
@@
       (reference "R2") (unit 1) (value "100k") (footprint "Resistors_THT:R_Axial_DIN0204_L3.6mm_D1.6mm_P7.62mm_Horizontal")
     )
+    (path "/95ef25aa-dac6-44d9-90a0-efd49308b704"
+      (reference "R3") (unit 1) (value "4.7k") (footprint "Resistors_THT:R_Axial_DIN0204_L3.6mm_D1.6mm_P7.62mm_Horizontal")
+    )
     (path "/b363d91d-fcd7-4752-acfe-6ce43382c232"
