File: Kicad/ZPE Atom controller/ZPE Atom controller.kicad_sch (KiCad schematic)
At the start: 33 parts, among them J1 50 ohm 21 turns, P1 CONN_01X18, P2 CONN_01X18, Q1 Q_PNP_ECB, Q2 IRF510, SW1 ON/OFF, T1 Transformer_SP_1S, U1 SSD1306, U2 LM7805_TO220

Commit message: Updated transisitor driver setup
Parts:
- removed R2: 100k, Resistors_THT:R_Axial_DIN0204_L3.6mm_D1.6mm_P7.62mm_Horizontal, symbol ZPE-test-3-small-board-only-rescue:R-device
- Q1: value Q_PNP_ECB -> 2N2222
Connections:
- net +12V: now also R1.1
- net GND: no longer R3.2
- net IO33: now also R3.1; no longer R1.2
- net at Q1.1 (E), Q2.1 (G): now also R1.2; no longer R3.1
- net at Q1.3 (B): now also R3.2; no longer R1.1
Other:
- moved on the sheet: L1, L2, L3, L4, R1, R3
Changed lines of the file:
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@@
   (junction (at 150.495 42.545) (diameter 0) (color 0 0 0 0)
   )
-  (junction (at 154.305 65.405) (diameter 0) (color 0 0 0 0)
-  )
   (junction (at 26.67 55.245) (diameter 0) (color 0 0 0 0)
   )
@@
     (stroke (width 0) (type default))
   )
-  (wire (pts (xy 150.495 65.405) (xy 154.305 65.405))
+  (wire (pts (xy 150.495 65.405) (xy 154.94 65.405))
     (stroke (width 0) (type default))
   )
@@
     (stroke (width 0) (type default))
   )
-  (wire (pts (xy 154.305 65.405) (xy 154.94 65.405))
-    (stroke (width 0) (type default))
-  )
   (wire (pts (xy 41.656 81.28) (xy 41.656 86.995))
     (stroke (width 0) (type default))
@@
   )
   (wire (pts (xy 209.55 133.985) (xy 209.55 128.905))
-    (stroke (width 0) (type default))
-  )
-  (wire (pts (xy 154.305 69.215) (xy 154.305 65.405))
     (stroke (width 0) (type default))
   )
@@
     (pin "1")
     (pin "2")
-  )
-  (symbol (lib_id "power:GND") (at 154.305 76.835 0) (unit 1)
-    (in_bom yes) (on_board yes) (fields_autoplaced)
-    (property "Reference" "#PWR08" (id 0) (at 154.305 83.185 0)
-      (effects (font (size 1.27 1.27)) hide)
-    )
-    (property "Value" "GND" (id 1) (at 154.305 81.915 0)
-      (effects (font (size 1.27 1.27)))
-    )
-    (property "Footprint" "" (id 2) (at 154.305 76.835 0)
-      (effects (font (size 1.27 1.27)) hide)
-    )
-    (property "Datasheet" "" (id 3) (at 154.305 76.835 0)
-      (effects (font (size 1.27 1.27)) hide)
-    )
-    (pin "1")
   )
   (symbol (lib_id "Hornbill-Devboard-rescue:+3.3V") (at 26.67 55.245 0) (unit 1)
@@
     (pin "2")
   )
-  (symbol (lib_id "ZPE-test-3-small-board-only-rescue:R-device") (at 154.305 73.025 0) (unit 1)
-    (in_bom yes) (on_board yes)
-    (property "Reference" "R3" (id 0) (at 153.035 67.945 0)
-      (effects (font (size 1.27 1.27)))
-    )
-    (property "Value" "4.7k" (id 1) (at 154.305 73.025 90)
-      (effects (font (size 1.27 1.27)))
-    )
-    (property "Footprint" "Resistors_THT:R_Axial_DIN0204_L3.6mm_D1.6mm_P7.62mm_Horizontal" (id 2) (at 152.527 73.025 90)
-      (effects (font (size 1.27 1.27)) hide)
-    )
-    (property "Datasheet" "" (id 3) (at 154.305 73.025 0)
+  (symbol (lib_id "ZPE-test-3-small-board-only-rescue:R-device") (at 133.985 77.47 90) (unit 1)
+    (in_bom yes) (on_board yes)
+    (property "Reference" "R3" (id 0) (at 133.985 74.93 90)
+      (effects (font (size 1.27 1.27)))
+    )
+    (property "Value" "4.7k" (id 1) (at 133.985 77.47 90)
+      (effects (font (size 1.27 1.27)))
+    )
+    (property "Footprint" "Resistors_THT:R_Axial_DIN0204_L3.6mm_D1.6mm_P7.62mm_Horizontal" (id 2) (at 133.985 79.248 90)
+      (effects (font (size 1.27 1.27)) hide)
+    )
+    (property "Datasheet" "" (id 3) (at 133.985 77.47 0)
       (effects (font (size 1.27 1.27)) hide)
     )
@@
     (pin "3")
   )
-  (symbol (lib_id "ZPE-test-3-small-board-only-rescue:R-device") (at 150.495 53.975 0) (unit 1)
-    (in_bom yes) (on_board yes)
-    (property "Reference" "R2" (id 0) (at 149.225 48.895 0)
-      (effects (font (size 1.27 1.27)))
-    )
-    (property "Value" "100k" (id 1) (at 150.495 53.975 90)
-      (effects (font (size 1.27 1.27)))
-    )
-    (property "Footprint" "Resistors_THT:R_Axial_DIN0204_L3.6mm_D1.6mm_P7.62mm_Horizontal" (id 2) (at 148.717 53.975 90)
-      (effects (font (size 1.27 1.27)) hide)
-    )
-    (property "Datasheet" "" (id 3) (at 150.495 53.975 0)
-      (effects (font (size 1.27 1.27)) hide)
-    )
-    (pin "1")
-    (pin "2")
-  )
   (symbol (lib_id "Hornbill-Devboard-rescue:+3.3V") (at 126.365 85.09 0) (unit 1)
     (in_bom yes) (on_board yes)
@@
       (effects (font (size 1.27 1.27)) (justify left))
     )
-    (property "Value" "Q_PNP_ECB" (id 1) (at 133.35 82.55 0)
+    (property "Value" "2N2222" (id 1) (at 149.225 73.025 0)
       (effects (font (size 1.27 1.27)) (justify left))
     )
@@
     (pin "2")
   )
-  (symbol (lib_id "ZPE-test-3-small-board-only-rescue:R-device") (at 133.985 77.47 270) (unit 1)
-    (in_bom yes) (on_board yes)
-    (property "Reference" "R1" (id 0) (at 139.065 76.2 90)
-      (effects (font (size 1.27 1.27)))
-    )
-    (property "Value" "1k" (id 1) (at 133.985 77.47 90)
-      (effects (font (size 1.27 1.27)))
-    )
-    (property "Footprint" "Resistors_THT:R_Axial_DIN0204_L3.6mm_D1.6mm_P7.62mm_Horizontal" (id 2) (at 133.985 75.692 90)
-      (effects (font (size 1.27 1.27)) hide)
-    )
-    (property "Datasheet" "" (id 3) (at 133.985 77.47 0)
+  (symbol (lib_id "ZPE-test-3-small-board-only-rescue:R-device") (at 150.495 53.975 0) (unit 1)
+    (in_bom yes) (on_board yes)
+    (property "Reference" "R1" (id 0) (at 149.225 48.895 90)
+      (effects (font (size 1.27 1.27)))
+    )
+    (property "Value" "1k" (id 1) (at 150.495 53.975 90)
+      (effects (font (size 1.27 1.27)))
+    )
+    (property "Footprint" "Resistors_THT:R_Axial_DIN0204_L3.6mm_D1.6mm_P7.62mm_Horizontal" (id 2) (at 148.717 53.975 90)
+      (effects (font (size 1.27 1.27)) hide)
+    )
+    (property "Datasheet" "" (id 3) (at 150.495 53.975 0)
       (effects (font (size 1.27 1.27)) hide)
     )
@@
       (reference "#PWR07") (unit 1) (value "GND") (footprint "")
     )
-    (path "/1a3c0592-bae7-4dc8-bfdf-de050749f428"
-      (reference "#PWR08") (unit 1) (value "GND") (footprint "")
-    )
     (path "/beea61b7-6b97-4cff-b7b6-f7b521c060b1"
       (reference "#PWR0101") (unit 1) (value "Earth") (footprint "")
@@
     )
     (path "/bba52ae1-2c60-4612-b640-b785ed4cdd7e"
-      (reference "Q1") (unit 1) (value "Q_PNP_ECB") (footprint "")
+      (reference "Q1") (unit 1) (value "2N2222") (footprint "")
     )
     (path "/eec6f1b0-e4aa-49f8-b4a3-e9424cd19e76"
@@
       (reference "R1") (unit 1) (value "1k") (footprint "Resistors_THT:R_Axial_DIN0204_L3.6mm_D1.6mm_P7.62mm_Horizontal")
     )
-    (path "/b55f6fd6-b5a9-46c1-9ccf-a9b9dbedb0ae"
-      (reference "R2") (unit 1) (value "100k") (footprint "Resistors_THT:R_Axial_DIN0204_L3.6mm_D1.6mm_P7.62mm_Horizontal")
-    )
     (path "/95ef25aa-dac6-44d9-90a0-efd49308b704"
