File: Kicad/2022-05-01 Test results/2022-05-01 Test results.kicad_sch (KiCad schematic)
At the start: 26 parts

Commit message: updated schematic
Other:
- note added: "2022-04-30 Freq zpe contoler out 114kHz over T1 4-3 700 volt sinus see screenshot of scope According to calculation a cap of 41 nf should resonate the L1 at 114kH L1 (6T) of T1 47uH L2 (12T) of T1 2.3mH"
- note removed: "Freq zpe contoler out 114kHz over T1 4-3 700 volt sinus see screenshot of scope"
Changed lines of the file:
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@@
     (effects (font (size 1.27 1.27)) (justify left bottom))
   )
-  (text "Freq zpe contoler out 114kHz\nover T1 4-3 700 volt sinus \nsee screenshot of scope"
-    (at 212.09 57.15 0)
+  (text "\n2022-04-30\nFreq zpe contoler out 114kHz\nover T1 4-3 700 volt sinus \nsee screenshot of scope\n\nAccording to calculation a cap of 41 nf should resonate the L1 at 114kH\n\nL1 (6T) of T1 47uH\nL2 (12T) of T1 2.3mH"
+    (at 211.455 67.945 0)
     (effects (font (size 1.27 1.27)) (justify left bottom))
   )
@@
     (effects (font (size 1.27 1.27)) (justify left))
     (property "Intersheetrefs" "${INTERSHEET_REFS}" (id 0) (at 200.5161 36.83 0)
-      (effects (font (size 1.27 1.27)) (justify left))
+      (effects (font (size 1.27 1.27)) (justify left) hide)
     )
   )
@@
     (effects (font (size 1.27 1.27)) (justify left))
     (property "Intersheetrefs" "${INTERSHEET_REFS}" (id 0) (at 228.1537 45.085 0)
-      (effects (font (size 1.27 1.27)) (justify left))
+      (effects (font (size 1.27 1.27)) (justify left) hide)
     )
   )
@@
     (effects (font (size 1.27 1.27)) (justify right))
     (property "Intersheetrefs" "${INTERSHEET_REFS}" (id 0) (at 48.1015 34.29 0)
-      (effects (font (size 1.27 1.27)) (justify right))
+      (effects (font (size 1.27 1.27)) (justify right) hide)
     )
   )

Commit message: move  workspace file
Parts:
- C1: renamed from U; value (none) -> 1NF 1.5K
- C11, C12, C13, C14, C15: renamed from U; value (none) -> 100nF; footprint (none) -> Capacitor_THT:C_Disc_D5.0mm_W2.5mm_P5.00mm
- C8: renamed from U; value (none) -> 1000uF
- DutyCycle1, Freq_super_fine1: renamed from U; value (none) -> 10k; footprint (none) -> Potentiometer_THT:Potentiometer_Piher_PC-16_Single_Vertical
- Freq_fine1, Freq_rough1, Resolution1: renamed from U; value (none) -> 10K; footprint (none) -> Potentiometer_THT:Potentiometer_Piher_PC-16_Single_Vertical
- IC1: renamed from U; value (none) -> TC4424AVPA; footprint (none) -> Package_DIP:DIP-8_W10.16mm
- L5: renamed from U; value (none) -> 150uH
- P1, P2: renamed from U; value (none) -> CONN_01X18; footprint (none) -> Connector_PinHeader_2.54mm:PinHeader_1x19_P2.54mm_Vertical
- Q2: renamed from U; value (none) -> IRF3205; footprint (none) -> Housings_SIP:SIP3_11.6x8.5mm
- R1: renamed from U; value (none) -> 470; footprint (none) -> Resistor_THT:R_Axial_DIN0207_L6.3mm_D2.5mm_P10.16mm_Horizontal
- R2: renamed from U; value (none) -> 1k; footprint (none) -> Resistor_THT:R_Axial_DIN0207_L6.3mm_D2.5mm_P10.16mm_Horizontal
- R6: renamed from U; value (none) -> 100; footprint (none) -> Potentiometer_THT:Potentiometer_Piher_T-16L_Single_Vertical_Hole
- SW2, SW3, SW4: renamed from U; value (none) -> SW_SPST
- T1: renamed from U; value (none) -> Transformer_SP_1S; footprint (none) -> Transformer_THT:Transformer_NF_ETAL_P1165
- U1: renamed from U; value (none) -> SSD1306; footprint (none) -> Package_TO_SOT_SMD:SOT-23-5
- U3: renamed from U; value 4009 -> 4049; footprint (none) -> Package_DIP:DIP-16_W7.62mm
